File: smart_pc_power_switch.kicad_sch (KiCad schematic)
At the start: 0 parts

Commit message: Add votlage divider for power sensor
Parts:
- added J1: Front Panel Connector, Connector_PinHeader_2.54mm:PinHeader_2x05_P2.54mm_Vertical, symbol Connector_Generic:Conn_02x05_Odd_Even
- added J2: INTERNAL_SPEAKER, Connector_PinHeader_2.54mm:PinHeader_1x04_P2.54mm_Vertical, symbol Connector_Generic:Conn_01x04
- added Q1, Q2: 2N3904, Package_TO_SOT_THT:TO-18-3_Lens, symbol Transistor_BJT:2N3904
- added R1, R2: 1k, Resistor_THT:R_Axial_DIN0204_L3.6mm_D1.6mm_P5.08mm_Horizontal, symbol Device:R_Small
- added R3: 6.8k, Resistor_THT:R_Axial_DIN0204_L3.6mm_D1.6mm_P5.08mm_Horizontal, symbol Device:R_Small
- added R4: 10k, Resistor_THT:R_Axial_DIN0204_L3.6mm_D1.6mm_P5.08mm_Horizontal, symbol Device:R_Small
- added SW1: PWR_SW, symbol Switch:SW_Push
- added SW2: RES_SW, symbol Switch:SW_Push
Connections:
- new net: Q1.2 (B), R1.2
- new net: Q2.2 (B), R2.2
- new net GND: J1.5 (Pin_5), J1.8 (Pin_8), Q1.1 (E), Q2.1 (E), R4.1, SW1.2, SW2.2
- new net GPIO0: R3.1, R4.2
- new net GPIO16: R2.1
- new net GPIO23: R1.1
- new net HDD+: J1.1 (Pin_1)
- new net HDD-: J1.3 (Pin_3)
- new net PLED+: J1.2 (Pin_2)
- new net PLED-: J1.4 (Pin_4)
- new net PWR+: J1.6 (Pin_6), Q1.3 (C), SW1.1
- new net RES+: J1.7 (Pin_7), Q2.3 (C), SW2.1
- new net SPKR_5V: J2.1 (Pin_1), R3.2
- no-connect marks 0 -> 2
Other:
- note added: "Use PC Speaker 5V rail to sense if PC is on or off"

Commit message: Initial PCB Drafted and Ordered
Parts:
- added J3: PWR_CONN, Connector_PinSocket_2.54mm:PinSocket_2x01_P2.54mm_Vertical_SMD, symbol Connector_Generic:Conn_01x02
- added J4: RES_CONN, Connector_PinSocket_2.54mm:PinSocket_2x01_P2.54mm_Vertical_SMD, symbol Connector_Generic:Conn_01x02
- added J5: SPKR_CONN, TestPoint:TestPoint_Pad_D2.5mm, symbol Connector_Generic:Conn_01x01
- added U1: XIAO-ESP32-S3-SMD, seeed_studio_xiao:XIAO-ESP32C6-SMD, symbol Seeed_Studio_XIAO_Series:XIAO-ESP32-C6-SMD
- J1, J2: now not fitted; now left out of the parts list
- Q1, Q2: footprint Package_TO_SOT_THT:TO-18-3_Lens -> Package_TO_SOT_THT:TO-92_Inline
- SW1, SW2: footprint (none) -> Button_Switch_THT:SW_PUSH_6mm_H5mm
Connections:
- net GPIO23 is gone; now on net GPIO0: R1.1
- net GND: now also J3.1 (Pin_1), J4.1 (Pin_1), U1.13 (GND), U1.16 (GND)
- net GPIO0: now also U1.1 (GPIO0_A0_D0); no longer R3.1, R4.2
- net PWR+: now also J3.2 (Pin_2)
- net RES+: now also J4.2 (Pin_2)
- net SPKR_5V: now also J5.1 (Pin_1)
- net GPIO16 renamed GPIO1
- net GPIO1: now also U1.2 (GPIO1_A1_D1)
- new net GPIO2: R3.1, R4.2, U1.3 (GPIO2_A2_D2)
- no-connect marks 2 -> 20
